File: AS077_DCF77_Empfaenger.brd (EAGLE design)
At the start: 160 x 100 mm, 82 parts, among them IC1 CA3130E, IC2 4093N, IC3 4538N, IC4 4093N, J1 Rückkopplung, J2 JUMPER_J5MM, J3 JUMPER_J5MM, Q1 34MM_PIEZO, T1 BC549C, T2 BF244A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

Commit message: * Renamed included library * Changed all references to new lib name
Parts:
- C1, C10, C16, C17, C19, C2, C4, C5, C6, C9: device 0027 DCF77-Empfänger:RCL_C050-024X044 -> AS077_DCF77_Empfaenger:RCL_C050-024X044
- C11, C13, C14, C15, C20, C7: device 0027 DCF77-Empfänger:RCL_C075-032X103 -> AS077_DCF77_Empfaenger:RCL_C075-032X103
- C12: device 0027 DCF77-Empfänger:E5-6 -> AS077_DCF77_Empfaenger:E5-6
- C18, C3: device 0027 DCF77-Empfänger:RCL_E5-10,5 -> AS077_DCF77_Empfaenger:RCL_E5-10,5
- C8: device 0027 DCF77-Empfänger:RCL_CTRIM808-BC7.5 -> AS077_DCF77_Empfaenger:RCL_CTRIM808-BC7.5
- D1, D2: device 0027 DCF77-Empfänger:DIODE_DO07 -> AS077_DCF77_Empfaenger:DIODE_DO07
- IC1: device 0027 DCF77-Empfänger:DIL08 -> AS077_DCF77_Empfaenger:DIL08
- IC2, IC4: device 0027 DCF77-Empfänger:DIL14 -> AS077_DCF77_Empfaenger:DIL14
- IC3: device 0027 DCF77-Empfänger:DIL16 -> AS077_DCF77_Empfaenger:DIL16
- J1, J2, J3: device 0027 DCF77-Empfänger:JUMPER_05 -> AS077_DCF77_Empfaenger:JUMPER_05
- LED1, LED2, LED3: device 0027 DCF77-Empfänger:LED_LED5MM -> AS077_DCF77_Empfaenger:LED_LED5MM
- PAD1, PAD10, PAD11, PAD12, PAD13, PAD14, PAD15, PAD16, PAD17, PAD18, PAD2, PAD3, PAD4, PAD5, PAD6, PAD7, PAD8, PAD9: device 0027 DCF77-Empfänger:WIREPAD_2.2/1.3 -> AS077_DCF77_Empfaenger:WIREPAD_2.2/1.3
- Q1: device 0027 DCF77-Empfänger:34MM_PIEZO_SCREW -> AS077_DCF77_Empfaenger:34MM_PIEZO_SCREW
- R1, R10, R11, R12, R13, R14, R15, R16, R19, R2, R20, R21, R4, R5, R6, R7, R8, R9: device 0027 DCF77-Empfänger:RCL_0207/5V -> AS077_DCF77_Empfaenger:RCL_0207/5V
- R17, R18, R22, R3: device 0027 DCF77-Empfänger:RCL_0207/15 -> AS077_DCF77_Empfaenger:RCL_0207/15
- R23: device 0027 DCF77-Empfänger:RCL_0207/10 -> AS077_DCF77_Empfaenger:RCL_0207/10
- T1, T2, T3, T4, T7: device 0027 DCF77-Empfänger:TO92_5.08 -> AS077_DCF77_Empfaenger:TO92_5.08
- T5, T6: device 0027 DCF77-Empfänger:TO92_2.54 -> AS077_DCF77_Empfaenger:TO92_2.54
- U$1: device 0027 DCF77-Empfänger:9V_BLOCK -> AS077_DCF77_Empfaenger:9V_BLOCK

Commit message: * More schematic and layout cleanup
Other:
- board text added: "Ant."
Changed lines of the file:
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@@
 <drawing>
 <settings>
-<setting alwaysvectorfont="no"/>
+<setting alwaysvectorfont="yes"/>
 <setting keepoldvectorfont="yes"/>
 <setting verticaltext="up"/>
 </settings>
-<grid distance="0.635" unitdist="mm" unit="mm" style="dots" multiple="1" display="yes" altdistance="0.05" altunitdist="mm" altunit="mm"/>
+<grid distance="2.5" unitdist="mm" unit="mm" style="dots" multiple="1" display="yes" altdistance="0.05" altunitdist="mm" altunit="mm"/>
 <layers>
 <layer number="1" name="Top" color="4" fill="1" visible="yes" active="yes"/>
@@
 <text x="35.56" y="17.78" size="2" layer="21" font="vector" ratio="15" align="center">B</text>
 <text x="38.1" y="12.7" size="2" layer="21" font="vector" ratio="15" align="center">C</text>
-<text x="12.7" y="63.5" size="2" layer="21" font="vector" ratio="15" align="center-right">Comp.</text>
-<text x="12.7" y="68.58" size="2" layer="21" font="vector" ratio="15" align="center-right">Masse</text>
-<text x="12.7" y="73.66" size="2" layer="21" font="vector" ratio="15" align="center-right">Masse</text>
-<text x="12.7" y="55.88" size="2" layer="21" font="vector" ratio="15" align="center-right">+</text>
+<text x="13.335" y="63.5" size="2" layer="21" font="vector" ratio="15" align="center-right">Comp.</text>
+<text x="13.335" y="68.58" size="2" layer="21" font="vector" ratio="15" align="center-right">Masse</text>
+<text x="13.335" y="73.66" size="2" layer="21" font="vector" ratio="15" align="center-right">Masse</text>
+<text x="13.335" y="55.88" size="2" layer="21" font="vector" ratio="15" align="center-right">+</text>
 <text x="68.58" y="34.925" size="2" layer="21" font="vector" ratio="15" align="center">"1"</text>
 <text x="78.74" y="34.925" size="2" layer="21" font="vector" ratio="15" align="center">"0"</text>
-<text x="116.84" y="33.655" size="2" layer="21" font="vector" ratio="15" align="center">G</text>
+<text x="116.84" y="33.02" size="2" layer="21" font="vector" ratio="15" align="center">G</text>
 <text x="118.745" y="50.8" size="2" layer="21" font="vector" ratio="15" align="center-left">+</text>
 <text x="121.92" y="45.085" size="2" layer="21" font="vector" ratio="15" align="center">P+</text>
@@
 <text x="35.56" y="46.355" size="2" layer="21" font="vector" ratio="15" align="center">F</text>
 <text x="50.8" y="48.895" size="2" layer="21" font="vector" ratio="15" align="center">E</text>
-<wire x1="10.16" y1="96.52" x2="148.59" y2="96.52" width="0.5" layer="21"/>
-<wire x1="148.59" y1="96.52" x2="148.59" y2="86.36" width="0.5" layer="21"/>
-<wire x1="148.59" y1="86.36" x2="135.255" y2="86.36" width="0.5" layer="21"/>
-<wire x1="135.255" y1="86.36" x2="62.23" y2="86.36" width="0.5" layer="21"/>
-<wire x1="62.23" y1="86.36" x2="10.16" y2="86.36" width="0.5" layer="21"/>
-<wire x1="10.16" y1="86.36" x2="10.16" y2="96.52" width="0.5" layer="21"/>
-<wire x1="137.16" y1="69.85" x2="137.16" y2="71.12" width="0.3" layer="21"/>
-<wire x1="137.16" y1="71.12" x2="135.255" y2="80.01" width="0.3" layer="21" curve="31.890792"/>
-<wire x1="135.255" y1="80.01" x2="135.255" y2="86.36" width="0.3" layer="21" curve="-63.781572"/>
-<wire x1="121.92" y1="80.01" x2="121.92" y2="81.28" width="0.3" layer="21"/>
-<wire x1="121.92" y1="81.28" x2="119.38" y2="83.82" width="0.3" layer="21" curve="90"/>
-<wire x1="119.38" y1="83.82" x2="64.77" y2="85.09" width="0.3" layer="21" curve="-2.66444"/>
-<wire x1="64.77" y1="85.09" x2="62.23" y2="86.36" width="0.3" layer="21" curve="-84.671157"/>
+<wire x1="10" y1="97.5" x2="150" y2="97.5" width="0.5" layer="21"/>
+<wire x1="150" y1="97.5" x2="150" y2="87.5" width="0.5" layer="21"/>
+<wire x1="150" y1="87.5" x2="10" y2="87.5" width="0.5" layer="21"/>
+<wire x1="10" y1="87.5" x2="10" y2="97.5" width="0.5" layer="21"/>
 <wire x1="1.27" y1="53.34" x2="158.75" y2="53.34" width="0.3" layer="22" style="longdash"/>
 <text x="42.545" y="5.08" size="2" layer="22" font="vector" ratio="12" rot="MR0" align="center">https://github.com/SebiR</text>
 <text x="146.05" y="55.88" size="1.5" layer="22" font="vector" ratio="10" rot="MR0" align="center">Analog</text>
 <text x="146.05" y="50.8" size="1.5" layer="22" font="vector" ratio="10" rot="MR0" align="center">Digital</text>
-<text x="80" y="91.44" size="3" layer="25" font="vector" ratio="15" align="center">Ferritantenne</text>
+<text x="80" y="92.5" size="2" layer="25" font="vector" ratio="15" align="center">Ferritantenne</text>
 <text x="142.24" y="27.94" size="3" layer="25" font="vector" ratio="15" align="center">Piezo-
 Element</text>
@@
 <wire x1="129.54" y1="11.43" x2="128.905" y2="6.985" width="0.8" layer="21" curve="-68.238658"/>
 <wire x1="128.905" y1="6.985" x2="128.27" y2="3.81" width="0.8" layer="21" curve="61.878983"/>
-<wire x1="126.15" y1="41.275" x2="125.73" y2="41.275" width="0.5" layer="21"/>
-<wire x1="125.73" y1="41.275" x2="124.46" y2="39.37" width="0.5" layer="21" curve="112.619825"/>
-<wire x1="124.46" y1="39.37" x2="123.19" y2="38.1" width="0.5" layer="21" curve="-135.239531"/>
-<wire x1="127.635" y1="44.45" x2="127" y2="44.45" width="0.5" layer="21"/>
-<wire x1="127" y1="44.45" x2="125.095" y2="43.18" width="0.5" layer="21" curve="67.380135"/>
-<wire x1="125.095" y1="43.18" x2="123.825" y2="42.545" width="0.5" layer="21" curve="-81.630218"/>
-<wire x1="123.825" y1="42.545" x2="123.19" y2="43.18" width="0.5" layer="21" curve="-61.500073"/>
-<wire x1="123.19" y1="43.18" x2="122.555" y2="43.18" width="0.5" layer="21" curve="151.50012"/>
 <text x="118.11" y="50.8" size="2" layer="22" font="vector" ratio="15" rot="MR180" align="center-left">BAT+</text>
 <text x="123.19" y="33.02" size="2" layer="22" font="vector" ratio="15" rot="MR180" align="center-left">BAT-</text>
 <text x="142.24" y="3.81" size="2" layer="21" font="vector" ratio="15" align="center">AUS</text>
 <text x="142.24" y="13.97" size="2" layer="21" font="vector" ratio="15" align="center">EIN</text>
+<text x="137.16" y="70.485" size="1.2" layer="21" font="vector" ratio="12" align="center">Ant.</text>
+<text x="121.92" y="76.835" size="1.2" layer="21" font="vector" ratio="12" align="center">Ant.</text>
 </plain>
 <attributes>
